Commit message: Fix namespacing base station

File: exomy_description/urdf/exomy_model.xacro (robot description, xacro)
@@ -1,10 +1,8 @@
 <?xml version="1.0" encoding="utf-8"?>
-<!-- This URDF was automatically created by SolidWorks to URDF Exporter! Originally created by Stephen Brawner (brawner@gmail.com)
-     Commit Version: 1.5.1-0-g916b5db  Build Version: 1.5.7152.31018
-     For more information, please see http://wiki.ros.org/sw_urdf_exporter -->
 <robot
-  name="exomy_model">
-  <link
-    name="base_link">
+  name="exomy_model" xmlns:xacro="http://www.ros.org/wiki/xacro">
+  <xacro:arg name="prefix" default=""/>
+  <link
+    name="$(arg prefix)base_link">
     <inertial>
       <origin
@@ -45,8 +43,8 @@
   </link>
   <link
-    name="base_footprint">
-  </link>
-  <joint
-    name="footprint_joint"
+    name="$(arg prefix)base_footprint">
+  </link>
+  <joint
+    name="$(arg prefix)footprint_joint"
     type="fixed">
     <origin
@@ -54,10 +52,10 @@
       rpy="0 0 0" />
     <parent
-      link="base_link" />
-    <child
-      link="base_footprint" />
-  </joint>
-  <link
-    name="MRB_link">
+      link="$(arg prefix)base_link" />
+    <child
+      link="$(arg prefix)base_footprint" />
+  </joint>
+  <link
+    name="$(arg prefix)MRB_link">
     <inertial>
       <origin
@@ -103,7 +101,7 @@
       rpy="1.5708 0 1.5708" />
     <parent
-      link="base_link" />
-    <child
-      link="MRB_link" />
+      link="$(arg prefix)base_link" />
+    <child
+      link="$(arg prefix)MRB_link" />
     <axis
       xyz="0 0 1" />
@@ -115,5 +113,5 @@
   </joint>
   <link
-    name="STR_LR_link">
+    name="$(arg prefix)STR_LR_link">
     <inertial>
       <origin
@@ -159,7 +157,7 @@
       rpy="0 -1.5708 -1.5708" />
     <parent
-      link="MRB_link" />
-    <child
-      link="STR_LR_link" />
+      link="$(arg prefix)MRB_link" />
+    <child
+      link="$(arg prefix)STR_LR_link" />
     <axis
       xyz="0 0 1" />
@@ -171,5 +169,5 @@
   </joint>
   <link
-    name="DRV_LR_link">
+    name="$(arg prefix)DRV_LR_link">
     <inertial>
       <origin
@@ -217,7 +215,7 @@
       rpy="-1.5708 0 0" />
     <parent
-      link="STR_LR_link" />
-    <child
-      link="DRV_LR_link" />
+      link="$(arg prefix)STR_LR_link" />
+    <child
+      link="$(arg prefix)DRV_LR_link" />
     <axis
       xyz="0 0 1" />
@@ -227,5 +225,5 @@
   </joint>
   <link
-    name="STR_RR_link">
+    name="$(arg prefix)STR_RR_link">
     <inertial>
       <origin
@@ -271,7 +269,7 @@
       rpy="0 -1.5708 -1.5708" />
     <parent
-      link="MRB_link" />
-    <child
-      link="STR_RR_link" />
+      link="$(arg prefix)MRB_link" />
+    <child
+      link="$(arg prefix)STR_RR_link" />
     <axis
       xyz="0 0 1" />
@@ -283,5 +281,5 @@
   </joint>
   <link
-    name="DRV_RR_link">
+    name="$(arg prefix)DRV_RR_link">
     <inertial>
       <origin
@@ -329,7 +327,7 @@
       rpy="-1.57079634175582 0 0" />
     <parent
-      link="STR_RR_link" />
-    <child
-      link="DRV_RR_link" />
+      link="$(arg prefix)STR_RR_link" />
+    <child
+      link="$(arg prefix)DRV_RR_link" />
     <axis
       xyz="0 0 1" />
@@ -339,5 +337,5 @@
   </joint>
   <link
-    name="RFB_link">
+    name="$(arg prefix)RFB_link">
     <inertial>
       <origin
@@ -383,7 +381,7 @@
       rpy="-1.5707963267949 0 0" />
     <parent
-      link="base_link" />
-    <child
-      link="RFB_link" />
+      link="$(arg prefix)base_link" />
+    <child
+      link="$(arg prefix)RFB_link" />
     <axis
       xyz="0 0 1" />
@@ -395,5 +393,5 @@
   </joint>
   <link
-    name="STR_RF_link">
+    name="$(arg prefix)STR_RF_link">
     <inertial>
       <origin
@@ -439,7 +437,7 @@
       rpy="1.5707963267949 0 -0.015893290716378" />
     <parent
-      link="RFB_link" />
-    <child
-      link="STR_RF_link" />
+      link="$(arg prefix)RFB_link" />
+    <child
+      link="$(arg prefix)STR_RF_link" />
     <axis
       xyz="0 0 1" />
@@ -451,5 +449,5 @@
   </joint>
   <link
-    name="DRV_RF_link">
+    name="$(arg prefix)DRV_RF_link">
     <inertial>
       <origin
@@ -497,7 +495,7 @@
       rpy="-1.5707963267949 0.015893290716378 0" />
     <parent
-      link="STR_RF_link" />
-    <child
-      link="DRV_RF_link" />
+      link="$(arg prefix)STR_RF_link" />
+    <child
+      link="$(arg prefix)DRV_RF_link" />
     <axis
       xyz="0 0 1" />
@@ -507,5 +505,5 @@
   </joint>
   <link
-    name="STR_RM_link">
+    name="$(arg prefix)STR_RM_link">
     <inertial>
       <origin
@@ -551,7 +549,7 @@
       rpy="1.5707963267949 0 -0.0158932907163782" />
     <parent
-      link="RFB_link" />
-    <child
-      link="STR_RM_link" />
+      link="$(arg prefix)RFB_link" />
+    <child
+      link="$(arg prefix)STR_RM_link" />
     <axis
       xyz="0 0 1" />
@@ -563,5 +561,5 @@
   </joint>
   <link
-    name="DRV_RM_link">
+    name="$(arg prefix)DRV_RM_link">
     <inertial>
       <origin
@@ -609,7 +607,7 @@
       rpy="-1.57079634175582 0.0158932907163779 0" />
     <parent
-      link="STR_RM_link" />
-    <child
-      link="DRV_RM_link" />
+      link="$(arg prefix)STR_RM_link" />
+    <child
+      link="$(arg prefix)DRV_RM_link" />
     <axis
       xyz="0 0 1" />
@@ -619,5 +617,5 @@
   </joint>
   <link
-    name="LFB_link">
+    name="$(arg prefix)LFB_link">
     <inertial>
       <origin
@@ -663,7 +661,7 @@
       rpy="-1.5707963267949 0 0" />
     <parent
-      link="base_link" />
-    <child
-      link="LFB_link" />
+      link="$(arg prefix)base_link" />
+    <child
+      link="$(arg prefix)LFB_link" />
     <axis
       xyz="0 0 1" />
@@ -675,5 +673,5 @@
   </joint>
   <link
-    name="STR_LF_link">
+    name="$(arg prefix)STR_LF_link">
     <inertial>
       <origin
@@ -719,7 +717,7 @@
       rpy="1.5707963267949 0 0" />
     <parent
-      link="LFB_link" />
-    <child
-      link="STR_LF_link" />
+      link="$(arg prefix)LFB_link" />
+    <child
+      link="$(arg prefix)STR_LF_link" />
     <axis
       xyz="0 0 1" />
@@ -731,5 +729,5 @@
   </joint>
   <link
-    name="DRV_LF_link">
+    name="$(arg prefix)DRV_LF_link">
     <inertial>
       <origin
@@ -777,7 +775,7 @@
       rpy="-1.5707963267949 0 0" />
     <parent
-      link="STR_LF_link" />
-    <child
-      link="DRV_LF_link" />
+      link="$(arg prefix)STR_LF_link" />
+    <child
+      link="$(arg prefix)DRV_LF_link" />
     <axis
       xyz="0 0 1" />
@@ -787,5 +785,5 @@
   </joint>
   <link
-    name="STR_LM_link">
+    name="$(arg prefix)STR_LM_link">
     <inertial>
       <origin
@@ -831,7 +829,7 @@
       rpy="1.5707963267949 0 0" />
     <parent
-      link="LFB_link" />
-    <child
-      link="STR_LM_link" />
+      link="$(arg prefix)LFB_link" />
+    <child
+      link="$(arg prefix)STR_LM_link" />
     <axis
       xyz="0 0 1" />
@@ -843,5 +841,5 @@
   </joint>
   <link
-    name="DRV_LM_link">
+    name="$(arg prefix)DRV_LM_link">
     <inertial>
       <origin
@@ -889,7 +887,7 @@
       rpy="-1.5707963415217 0 0" />
     <parent
-      link="STR_LM_link" />
-    <child
-      link="DRV_LM_link" />
+      link="$(arg prefix)STR_LM_link" />
+    <child
+      link="$(arg prefix)DRV_LM_link" />
     <axis
       xyz="0 0 1" />
@@ -899,5 +897,5 @@
   </joint>
   <link
-    name="head_link">
+    name="$(arg prefix)head_link">
     <inertial>
       <origin
@@ -943,12 +941,12 @@
       rpy="1.5707963267949 0 1.5707963267949" />
     <parent
-      link="base_link" />
-    <child
-      link="head_link" />
+      link="$(arg prefix)base_link" />
+    <child
+      link="$(arg prefix)head_link" />
     <axis
       xyz="0 0 0" />
   </joint>
   <link
-    name="eyewhite_link">
+    name="$(arg prefix)eyewhite_link">
     <inertial>
       <origin
@@ -994,12 +992,12 @@
       rpy="0 0 0" />
     <parent
-      link="head_link" />
-    <child
-      link="eyewhite_link" />
+      link="$(arg prefix)head_link" />
+    <child
+      link="$(arg prefix)eyewhite_link" />
     <axis
       xyz="0 0 0" />
   </joint>
   <link
-    name="pupil_left_link">
+    name="$(arg prefix)pupil_left_link">
     <inertial>
       <origin
@@ -1045,12 +1043,12 @@
       rpy="0 0 0" />
     <parent
-      link="eyewhite_link" />
-    <child
-      link="pupil_left_link" />
-    <axis
-      xyz="0 0 1" />
-  </joint>
-  <link
-    name="pupil_right_link">
+      link="$(arg prefix)eyewhite_link" />
+    <child
+      link="$(arg prefix)pupil_left_link" />
+    <axis
+      xyz="0 0 1" />
+  </joint>
+  <link
+    name="$(arg prefix)pupil_right_link">
     <inertial>
       <origin
@@ -1096,7 +1094,7 @@
       rpy="0 0 0" />
     <parent
-      link="eyewhite_link" />
-    <child
-      link="pupil_right_link" />
+      link="$(arg prefix)eyewhite_link" />
+    <child
+      link="$(arg prefix)pupil_right_link" />
     <axis
       xyz="0 0 1" />
@@ -1105,5 +1103,5 @@
   </joint>
   <link
-    name="camera">
+    name="$(arg prefix)camera">
     <inertial>
       <origin
@@ -1149,12 +1147,12 @@
       rpy="-0.785398 0 3.14159" />
     <parent
-      link="head_link" />
-    <child
-      link="camera" />
+      link="$(arg prefix)head_link" />
+    <child
+      link="$(arg prefix)camera" />
     <axis
       xyz="0 0 0" />
   </joint>
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
Commit message: tf namespacing

File: exomy_description/urdf/exomy_model.xacro (robot description, xacro)
@@ -2,7 +2,6 @@
 <robot
   name="exomy_model" xmlns:xacro="http://www.ros.org/wiki/xacro">
-  <xacro:arg name="prefix" default=""/>
-  <link
-    name="$(arg prefix)base_link">
+  <link
+    name="base_link">
     <inertial>
       <origin
@@ -43,8 +42,8 @@
   </link>
   <link
-    name="$(arg prefix)base_footprint">
-  </link>
-  <joint
-    name="$(arg prefix)footprint_joint"
+    name="base_footprint">
+  </link>
+  <joint
+    name="footprint_joint"
     type="fixed">
     <origin
@@ -52,10 +51,10 @@
       rpy="0 0 0" />
     <parent
-      link="$(arg prefix)base_link" />
-    <child
-      link="$(arg prefix)base_footprint" />
-  </joint>
-  <link
-    name="$(arg prefix)MRB_link">
+      link="base_link" />
+    <child
+      link="base_footprint" />
+  </joint>
+  <link
+    name="MRB_link">
     <inertial>
       <origin
@@ -101,7 +100,7 @@
       rpy="1.5708 0 1.5708" />
     <parent
-      link="$(arg prefix)base_link" />
-    <child
-      link="$(arg prefix)MRB_link" />
+      link="base_link" />
+    <child
+      link="MRB_link" />
     <axis
       xyz="0 0 1" />
@@ -113,5 +112,5 @@
   </joint>
   <link
-    name="$(arg prefix)STR_LR_link">
+    name="STR_LR_link">
     <inertial>
       <origin
@@ -157,7 +156,7 @@
       rpy="0 -1.5708 -1.5708" />
     <parent
-      link="$(arg prefix)MRB_link" />
-    <child
-      link="$(arg prefix)STR_LR_link" />
+      link="MRB_link" />
+    <child
+      link="STR_LR_link" />
     <axis
       xyz="0 0 1" />
@@ -169,5 +168,5 @@
   </joint>
   <link
-    name="$(arg prefix)DRV_LR_link">
+    name="DRV_LR_link">
     <inertial>
       <origin
@@ -215,7 +214,7 @@
       rpy="-1.5708 0 0" />
     <parent
-      link="$(arg prefix)STR_LR_link" />
-    <child
-      link="$(arg prefix)DRV_LR_link" />
+      link="STR_LR_link" />
+    <child
+      link="DRV_LR_link" />
     <axis
       xyz="0 0 1" />
@@ -225,5 +224,5 @@
   </joint>
   <link
-    name="$(arg prefix)STR_RR_link">
+    name="STR_RR_link">
     <inertial>
       <origin
@@ -269,7 +268,7 @@
       rpy="0 -1.5708 -1.5708" />
     <parent
-      link="$(arg prefix)MRB_link" />
-    <child
-      link="$(arg prefix)STR_RR_link" />
+      link="MRB_link" />
+    <child
+      link="STR_RR_link" />
     <axis
       xyz="0 0 1" />
@@ -281,5 +280,5 @@
   </joint>
   <link
-    name="$(arg prefix)DRV_RR_link">
+    name="DRV_RR_link">
     <inertial>
       <origin
@@ -327,7 +326,7 @@
       rpy="-1.57079634175582 0 0" />
     <parent
-      link="$(arg prefix)STR_RR_link" />
-    <child
-      link="$(arg prefix)DRV_RR_link" />
+      link="STR_RR_link" />
+    <child
+      link="DRV_RR_link" />
     <axis
       xyz="0 0 1" />
@@ -337,5 +336,5 @@
   </joint>
   <link
-    name="$(arg prefix)RFB_link">
+    name="RFB_link">
     <inertial>
       <origin
@@ -381,7 +380,7 @@
       rpy="-1.5707963267949 0 0" />
     <parent
-      link="$(arg prefix)base_link" />
-    <child
-      link="$(arg prefix)RFB_link" />
+      link="base_link" />
+    <child
+      link="RFB_link" />
     <axis
       xyz="0 0 1" />
@@ -393,5 +392,5 @@
   </joint>
   <link
-    name="$(arg prefix)STR_RF_link">
+    name="STR_RF_link">
     <inertial>
       <origin
@@ -437,7 +436,7 @@
       rpy="1.5707963267949 0 -0.015893290716378" />
     <parent
-      link="$(arg prefix)RFB_link" />
-    <child
-      link="$(arg prefix)STR_RF_link" />
+      link="RFB_link" />
+    <child
+      link="STR_RF_link" />
     <axis
       xyz="0 0 1" />
@@ -449,5 +448,5 @@
   </joint>
   <link
-    name="$(arg prefix)DRV_RF_link">
+    name="DRV_RF_link">
     <inertial>
       <origin
@@ -495,7 +494,7 @@
       rpy="-1.5707963267949 0.015893290716378 0" />
     <parent
-      link="$(arg prefix)STR_RF_link" />
-    <child
-      link="$(arg prefix)DRV_RF_link" />
+      link="STR_RF_link" />
+    <child
+      link="DRV_RF_link" />
     <axis
       xyz="0 0 1" />
@@ -505,5 +504,5 @@
   </joint>
   <link
-    name="$(arg prefix)STR_RM_link">
+    name="STR_RM_link">
     <inertial>
       <origin
@@ -549,7 +548,7 @@
       rpy="1.5707963267949 0 -0.0158932907163782" />
     <parent
-      link="$(arg prefix)RFB_link" />
-    <child
-      link="$(arg prefix)STR_RM_link" />
+      link="RFB_link" />
+    <child
+      link="STR_RM_link" />
     <axis
       xyz="0 0 1" />
@@ -561,5 +560,5 @@
   </joint>
   <link
-    name="$(arg prefix)DRV_RM_link">
+    name="DRV_RM_link">
     <inertial>
       <origin
@@ -607,7 +606,7 @@
       rpy="-1.57079634175582 0.0158932907163779 0" />
     <parent
-      link="$(arg prefix)STR_RM_link" />
-    <child
-      link="$(arg prefix)DRV_RM_link" />
+      link="STR_RM_link" />
+    <child
+      link="DRV_RM_link" />
     <axis
       xyz="0 0 1" />
@@ -617,5 +616,5 @@
   </joint>
   <link
-    name="$(arg prefix)LFB_link">
+    name="LFB_link">
     <inertial>
       <origin
@@ -661,7 +660,7 @@
       rpy="-1.5707963267949 0 0" />
     <parent
-      link="$(arg prefix)base_link" />
-    <child
-      link="$(arg prefix)LFB_link" />
+      link="base_link" />
+    <child
+      link="LFB_link" />
     <axis
       xyz="0 0 1" />
@@ -673,5 +672,5 @@
   </joint>
   <link
-    name="$(arg prefix)STR_LF_link">
+    name="STR_LF_link">
     <inertial>
       <origin
@@ -717,7 +716,7 @@
       rpy="1.5707963267949 0 0" />
     <parent
-      link="$(arg prefix)LFB_link" />
-    <child
-      link="$(arg prefix)STR_LF_link" />
+      link="LFB_link" />
+    <child
+      link="STR_LF_link" />
     <axis
       xyz="0 0 1" />
@@ -729,5 +728,5 @@
   </joint>
   <link
-    name="$(arg prefix)DRV_LF_link">
+    name="DRV_LF_link">
     <inertial>
       <origin
@@ -775,7 +774,7 @@
       rpy="-1.5707963267949 0 0" />
     <parent
-      link="$(arg prefix)STR_LF_link" />
-    <child
-      link="$(arg prefix)DRV_LF_link" />
+      link="STR_LF_link" />
+    <child
+      link="DRV_LF_link" />
     <axis
       xyz="0 0 1" />
@@ -785,5 +784,5 @@
   </joint>
   <link
-    name="$(arg prefix)STR_LM_link">
+    name="STR_LM_link">
     <inertial>
       <origin
@@ -829,7 +828,7 @@
       rpy="1.5707963267949 0 0" />
     <parent
-      link="$(arg prefix)LFB_link" />
-    <child
-      link="$(arg prefix)STR_LM_link" />
+      link="LFB_link" />
+    <child
+      link="STR_LM_link" />
     <axis
       xyz="0 0 1" />
@@ -841,5 +840,5 @@
   </joint>
   <link
-    name="$(arg prefix)DRV_LM_link">
+    name="DRV_LM_link">
     <inertial>
       <origin
@@ -887,7 +886,7 @@
       rpy="-1.5707963415217 0 0" />
     <parent
-      link="$(arg prefix)STR_LM_link" />
-    <child
-      link="$(arg prefix)DRV_LM_link" />
+      link="STR_LM_link" />
+    <child
+      link="DRV_LM_link" />
     <axis
       xyz="0 0 1" />
@@ -897,5 +896,5 @@
   </joint>
   <link
-    name="$(arg prefix)head_link">
+    name="head_link">
     <inertial>
       <origin
@@ -941,12 +940,12 @@
       rpy="1.5707963267949 0 1.5707963267949" />
     <parent
-      link="$(arg prefix)base_link" />
-    <child
-      link="$(arg prefix)head_link" />
+      link="base_link" />
+    <child
+      link="head_link" />
     <axis
       xyz="0 0 0" />
   </joint>
   <link
-    name="$(arg prefix)eyewhite_link">
+    name="eyewhite_link">
     <inertial>
       <origin
@@ -992,12 +991,12 @@
       rpy="0 0 0" />
     <parent
-      link="$(arg prefix)head_link" />
-    <child
-      link="$(arg prefix)eyewhite_link" />
+      link="head_link" />
+    <child
+      link="eyewhite_link" />
     <axis
       xyz="0 0 0" />
   </joint>
   <link
-    name="$(arg prefix)pupil_left_link">
+    name="pupil_left_link">
     <inertial>
       <origin
@@ -1043,12 +1042,12 @@
       rpy="0 0 0" />
     <parent
-      link="$(arg prefix)eyewhite_link" />
-    <child
-      link="$(arg prefix)pupil_left_link" />
-    <axis
-      xyz="0 0 1" />
-  </joint>
-  <link
-    name="$(arg prefix)pupil_right_link">
+      link="eyewhite_link" />
+    <child
+      link="pupil_left_link" />
+    <axis
+      xyz="0 0 1" />
+  </joint>
+  <link
+    name="pupil_right_link">
     <inertial>
       <origin
@@ -1094,7 +1093,7 @@
       rpy="0 0 0" />
     <parent
-      link="$(arg prefix)eyewhite_link" />
-    <child
-      link="$(arg prefix)pupil_right_link" />
+      link="eyewhite_link" />
+    <child
+      link="pupil_right_link" />
     <axis
       xyz="0 0 1" />
@@ -1103,5 +1102,5 @@
   </joint>
   <link
-    name="$(arg prefix)camera">
+    name="camera">
     <inertial>
       <origin
@@ -1147,12 +1146,12 @@
       rpy="-0.785398 0 3.14159" />
     <parent
-      link="$(arg prefix)head_link" />
-    <child
-      link="$(arg prefix)camera" />
+      link="head_link" />
+    <child
+      link="camera" />
     <axis
       xyz="0 0 0" />
   </joint>
   <link
-    name="$(arg prefix)hat_link">
+    name="hat_link">
     <inertial>
       <origin
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