Commit message: Add arducam and laserscan nodes

File: exomy_description/urdf/exomy_model.urdf (robot description, URDF)
Before this commit: robot exomy_model, 23 links, 22 joints
Links:
- removed link cam_link
- added link camera, mass 0.00115745344893818; visual mesh filename=package://exomy_description/meshes/cam_link.STL
Joints:
- joint cam_joint: child cam_link -> camera

Commit message: Corrects camera frame rotation

File: exomy_description/urdf/exomy_model.urdf (robot description, URDF)
Before this commit: robot exomy_model, 23 links, 22 joints
Joints:
- joint cam_joint: origin xyz=9.42151964158384E-05 0.00215468910946459 0.035 rpy=0 -0.7853982 1.5707963267949 -> xyz=9.42151964158384E-05 0.00215468910946459 0.035 rpy=-0.785398 0 3.14159

Commit message: Set arducam and laserscan params

File: exomy_description/urdf/exomy_model.urdf (robot description, URDF)
Before this commit: robot exomy_model, 23 links, 22 joints
Links:
- added link base_footprint
Joints:
- added joint footprint_joint: type fixed, parent base_link, child base_footprint, origin xyz=0 0 -0.1 rpy=0 0 0

Commit message: Fix imu and odom stuff!

File: exomy_description/urdf/exomy_model.urdf (robot description, URDF)
Before this commit: robot exomy_model, 25 links, 24 joints
Links:
- added link imu
Joints:
- added joint imu_joint: type fixed, parent base_link, child imu, origin xyz=0 0 0 rpy=0 0 0

File: exomy_description/urdf/exomy_model.xacro (robot description, xacro)
@@ -1152,4 +1152,10 @@
       xyz="0 0 0" />
   </joint>
+  <link name="imu"/>
+    <joint name="imu_joint" type="fixed">
+      <parent link="base_link" />
+      <child link="imu" />
+      <origin rpy="0 0 0" xyz="0 0 0" />
+    </joint>
   <link
     name="hat_link">
